File: Hardware/POW_SUPPLY/PowerSupplySA.sch (KiCad schematic (older format))
At the start: 18 parts, among them P1 CONN_01X02, Q1 Q_PMOS_GSD, Q2 Q_PNP_BCE, Q3 Q_PNP_BCE, U1 LM1117ADJ

Commit message: Shematic merger and stuff
Parts:
- P1: symbol Conn_01x02 -> CONN_01X02
Other:
- moved on the sheet: C1, C2, C3, C4, C5, C6, C7, D1, L1, L2, Q1, Q2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
