File: Hardware/CPU_Board/CPU_Board.sch (KiCad schematic (older format))
At the start: 76 parts, among them P1 CONN_01X02, P10 CONN_01X04, P2 USB_B, P3 CONN_01X06, P4 CONN_01X01, P5 CONN_01X01, P6 CONN_01X01, P7 CONN_01X01, P8 CONN_01X01, P9 CONN_01X01, Q1 Q_PMOS_GSD, Q2 Q_PNP_BCE, Q3 Q_PNP_BCE, Q4 N-Channel, Q5 P-Channel, U1 STM32F411RETx, U2 FT232RL, U3 LM1117ADJ, U4 6N136, U5 SPBTLE-RF, U6 A2235-H, U7 LSM303AGR, U8 LSM6DSL, U9 INA128, Y1 8MHz

Commit message: PCB v0.1.0
* Changed components to SMD
* Added Measurement nodes for all datalines
* Designed PCB (Rather big now, only a first edition!)
* "Fixed" fucked up power flags
Parts:
- removed U4: 6N136, Housings_DIP:DIP-8_W7.62mm_Socket, symbol 6N136
- added P10, P12, P14: CONN_01X03, Pin_Headers:Pin_Header_Straight_1x03_Pitch2.54mm, symbol CONN_01X03
- added P11, P13: CONN_01X01, Pin_Headers:Pin_Header_Straight_1x01_Pitch2.54mm, symbol CONN_01X01
- added P5, P6, P7, P8: CONN_01X02, Pin_Headers:Pin_Header_Straight_1x02_Pitch2.54mm, symbol CONN_01X02
- added P9: CONN_01X06, Pin_Headers:Pin_Header_Straight_1x06_Pitch2.54mm, symbol CONN_01X06
- added R19, R21, R22: 0C, Resistors_ThroughHole:R_Axial_DIN0204_L3.6mm_D1.6mm_P1.90mm_Vertical, symbol R_Small
- added R20: 0C, Resistors_ThroughHole:R_Axial_DIN0204_L3.6mm_D1.6mm_P2.54mm_Vertical, symbol R_Small
- C1, C18, C2, C20, C3, C6, C8: footprint Capacitors_ThroughHole:C_Axial_L3.8mm_D2.6mm_P7.50mm_Horizontal -> Capacitors_SMD:C_0805_HandSoldering
- C10: renamed from C14; footprint Capacitors_ThroughHole:C_Axial_L3.8mm_D2.6mm_P7.50mm_Horizontal -> Capacitors_SMD:C_0805_HandSoldering
- C11: renamed from C9; footprint Capacitors_ThroughHole:C_Axial_L3.8mm_D2.6mm_P7.50mm_Horizontal -> Capacitors_SMD:C_0805_HandSoldering
- C12: renamed from C15; footprint Capacitors_ThroughHole:C_Axial_L3.8mm_D2.6mm_P7.50mm_Horizontal -> Capacitors_SMD:C_0805_HandSoldering
- C13: renamed from C10; footprint Capacitors_ThroughHole:C_Axial_L3.8mm_D2.6mm_P7.50mm_Horizontal -> Capacitors_SMD:C_0805_HandSoldering
- C14: renamed from C16; footprint Capacitors_ThroughHole:C_Axial_L3.8mm_D2.6mm_P7.50mm_Horizontal -> Capacitors_SMD:C_0805_HandSoldering
- C15: renamed from C17; footprint Capacitors_ThroughHole:C_Axial_L3.8mm_D2.6mm_P7.50mm_Horizontal -> Capacitors_SMD:C_0805_HandSoldering
- C16: renamed from C12; footprint Capacitors_ThroughHole:C_Axial_L3.8mm_D2.6mm_P7.50mm_Horizontal -> Capacitors_SMD:C_0805_HandSoldering
- C17: renamed from C13; footprint Capacitors_ThroughHole:CP_Axial_L10.0mm_D4.5mm_P15.00mm_Horizontal -> Capacitors_SMD:CP_Elec_5x5.3
- C19, C7: footprint Capacitors_ThroughHole:CP_Axial_L10.0mm_D4.5mm_P15.00mm_Horizontal -> Capacitors_SMD:CP_Elec_5x5.3
- C21: renamed from C23; footprint Capacitors_ThroughHole:C_Axial_L3.8mm_D2.6mm_P7.50mm_Horizontal -> Capacitors_SMD:C_0805_HandSoldering
- C22: renamed from C24; footprint Capacitors_ThroughHole:C_Axial_L3.8mm_D2.6mm_P7.50mm_Horizontal -> Capacitors_SMD:C_0805_HandSoldering
- C23: renamed from C25; footprint Capacitors_ThroughHole:C_Axial_L3.8mm_D2.6mm_P7.50mm_Horizontal -> Capacitors_SMD:C_0805_HandSoldering
- C24: renamed from C26; footprint Capacitors_ThroughHole:CP_Axial_L10.0mm_D4.5mm_P15.00mm_Horizontal -> Capacitors_SMD:CP_Elec_5x5.3
- C25: renamed from C27; footprint Capacitors_ThroughHole:C_Axial_L3.8mm_D2.6mm_P7.50mm_Horizontal -> Capacitors_SMD:C_0805_HandSoldering
- C26: renamed from C28; footprint Capacitors_ThroughHole:C_Axial_L3.8mm_D2.6mm_P7.50mm_Horizontal -> Capacitors_SMD:C_0805_HandSoldering
- C27: renamed from C29; footprint Capacitors_ThroughHole:C_Axial_L3.8mm_D2.6mm_P7.50mm_Horizontal -> Capacitors_SMD:C_0805_HandSoldering
- C28: renamed from C30; footprint Capacitors_ThroughHole:C_Axial_L3.8mm_D2.6mm_P7.50mm_Horizontal -> Capacitors_SMD:C_0805_HandSoldering
- C29: renamed from C21; footprint Capacitors_ThroughHole:C_Axial_L3.8mm_D2.6mm_P7.50mm_Horizontal -> Capacitors_SMD:C_0805_HandSoldering
- C4, C5: footprint Capacitors_ThroughHole:CP_Axial_L10.0mm_D4.5mm_P15.00mm_Horizontal -> Capacitors_SMD:CP_Elec_4x5.3
- C9: renamed from C11; footprint Capacitors_ThroughHole:CP_Axial_L10.0mm_D4.5mm_P15.00mm_Horizontal -> Capacitors_SMD:CP_Elec_4x5.3
- D1: footprint Diodes_ThroughHole:D_5W_P5.08mm_Vertical_AnodeUp -> Diodes_SMD:D_SOD-323
- L2, L3: footprint Connectors:bornier2 -> Inductors:INDUCTOR_V
- R1, R10, R11, R12, R13, R15, R16, R17, R18, R2, R3, R4, R5, R6, R7, R8, R9: footprint Resistors_ThroughHole:R_Axial_DIN0204_L3.6mm_D1.6mm_P5.08mm_Horizontal -> Resistors_SMD:R_0805_HandSoldering
- U5: renamed from U6; footprint FOOTPRINTS:A2235-H -> FOOTPRINTS:A2235-H_Handsolder
- renumbered P4 to P15, P5 to P16, P6 to P17, P7 to P18, P8 to P19, P9 to P20, P10 to P3, P3 to P4, U5 to U4, U7 to U6, U8 to U7, U9 to U8
Connections:
- net +3.3VADC: now also P14.3 (P3)
- net +3V3: now also P10.3 (P3)
- net +5V: now also P10.1 (P1)
- net +5VA: now also P14.1 (P1)
- net BT_10_PA1: now also P9.5 (P5)
- net BT_11_PA8: now also P9.1 (P1)
- net BT_5_PA0: now also P9.6 (P6)
- net BT_7_PB3: now also P9.4 (P4)
- net BT_8_PA6: now also P9.2 (P2)
- net BT_9_PA7: now also P9.3 (P3)
- net GND: now also P2.4 (GND), P2.5 (shield), P10.2 (P2); no longer P2.1 (VBUS)
- net GNDA: now also U1.25 (PC5/ADC1_IN15), P14.2 (P2)
- net GPS_RX: now also R21.2, R22.1
- net GPS_TOGGLE: now also P11.1 (P1)
- net GPS_TX: now also R19.1, R20.2
- net GPS_USART_RX: now also P7.2 (P2), R19.2, R22.2
- net GPS_USART_TX: now also P7.1 (P1), R20.1, R21.1
- net IMU_I2C_CL: now also U1.58 (I2C1_SCL/TIM4_CH1/USART1_TX/PB6), P5.2 (P2); no longer U1.41 (I2C3_SCL/RCC_MCO_1/SDIO_D1/TIM1_CH1/USART1_CK/USB_OTG_FS_SOF/PA8)
- net IMU_I2C_DA: now also U1.59 (I2C1_SDA/SDIO_D0/TIM4_CH2/USART1_RX/PB7), P5.1 (P1); no longer U1.56 (I2C3_SDA/I2S3_ext_SD/SDIO_D0/SPI1_MISO/SPI3_MISO/SYS_JTRST/TIM3_CH1/PB4)
- net LSM303AGR_INT_1_XL: now also P12.3 (P3)
- net LSM303AGR_INT_2_XL: now also P12.2 (P2)
- net LSM303AGR_INT_MAG: now also P12.1 (P1)
- net LSM6DSL_INT1: now also P8.2 (P2)
- net LSM6DSL_INT2: now also P8.1 (P1)
- net Load_cell_amp: now also U1.24 (PC4/ADC1_IN14), P13.1 (P1); no longer U1.8 (PC0/ADC1_IN10)
- net USB_USART_RX: now also P6.2 (P2)
- net USB_USART_TX: now also P6.1 (P1)
- net at U2.15 (USBDP): now also P2.3 (D+); no longer P2.2 (D-)
- net at U2.16 (USBDM): now also P2.2 (D-); no longer P2.3 (D+)
- net at L1.1: now also P2.1 (VBUS); no longer P2.4 (GND)
- no-connect marks 83 -> 75
Other:
- note added: "IMU 1 interrupt pins"
- note added: "IMU 2 interrupt pins"
- note added: "Measurement\nNodes Analog\nPower Pins"
- note added: "Measurement\nNodes BT-LE"
- note added: "Measurement\nNodes Digital\nPower Pins"
- note added: "Measurement\nNodes GPS"
- note added: "Measurement\nNodes IMU\n1: (Magneto & Acc.)\n2: (Gyro & Acc.)"
- note added: "Measurement\nNodes MCU"
- note added: "Measurement\nNodes USB"
- note added: "Measurement\nNodes\nLoad Cell"
- note added: "Meta circuitry\n(Measurement nodes & Mounting)"
- note added: "Modules"
- note added: "Power Flags"
- note added: "Reset\nSPI_MISO\nSPI_MOSI\nSPI_CLK\nSPI_CS\nSPI_IRQ"
- note added: "Toggle signal\nGPS"
- note removed: "Measurement\nNodes"
- note removed: "OctoAwesome"
- moved on the sheet: C1, C10, C11, C12, C13, C14, C15, C16, C17, C18, C19, C2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

Commit message: PCB_Design v0.2
Added, changed and stuff.
Libraries and stuff.
Looks like shit, but it should work.
Will check later and then send gerbers.
Parts:
- removed R19, R22: 0C, Resistors_ThroughHole:R_Axial_DIN0204_L3.6mm_D1.6mm_P1.90mm_Vertical, symbol R_Small
- removed R20: 0C, Resistors_ThroughHole:R_Axial_DIN0204_L3.6mm_D1.6mm_P2.54mm_Vertical, symbol R_Small
- added C27: 100n, Capacitors_SMD:C_0805_HandSoldering, symbol C
- added D2: D_Photo, Opto-Devices:PhotoDiode_SFH205, symbol D_Photo
- added R15: 1k, Resistors_SMD:R_0805_HandSoldering, symbol R
- added R18: 10k, Resistors_SMD:R_0805_HandSoldering, symbol R
- added U8: MCDTS2-4N, Buttons_Switches_SMD:SW_SPST_PTS645, symbol CHERRY-MX
- R21: value 0C -> 0R; footprint Resistors_ThroughHole:R_Axial_DIN0204_L3.6mm_D1.6mm_P1.90mm_Vertical -> Resistors_ThroughHole:R_Axial_DIN0204_L3.6mm_D1.6mm_P5.08mm_Horizontal
- U6: symbol LSM303AGR -> LSM303Cx
- renumbered C11 to C10, C10 to C11, C16 to C15, C15 to C16, C27 to C28, C28 to C29, C29 to C30, R15 to R16, R16 to R17, R17 to R19, R18 to R20, U8 to U9
Connections:
- net GPS_USART_RX is gone; now on net GPS_TX: P7.2 (P2), U1.43 (I2S5_SD/SPI5_MOSI/TIM1_CH3/USART1_RX/USB_OTG_FS_ID/PA10)
- net LSM303AGR_INT_MAG is gone; now on net 303C_I_MAG: P12.1 (P1), U6.7 (INT_MAG)
- net +3V3: now also D2.1 (K), R18.2
- net BT_10_PA1: now also U1.15 (ADC1_IN1/I2S4_SD/SPI4_MOSI/TIM2_CH2/TIM5_CH2/USART2_RTS/PA1)
- net BT_11_PA8: now also U1.41 (I2C3_SCL/RCC_MCO_1/SDIO_D1/TIM1_CH1/USART1_CK/USB_OTG_FS_SOF/PA8)
- net BT_5_PA0: now also U1.14 (ADC1_IN0/SYS_WKUP/TIM2_CH1/TIM2_ETR/TIM5_CH1/USART2_CTS/PA0)
- net BT_7_PB3: now also P9.3 (P3), U1.55 (I2C2_SDA/I2S1_CK/I2S3_CK/SPI1_SCK/SPI3_SCK/SYS_JTDO-SWO/TIM2_CH2/USART1_RX/PB3); no longer P9.4 (P4)
- net BT_8_PA6: now also U1.22 (ADC1_IN6/I2S2_MCK/SDIO_CMD/SPI1_MISO/TIM1_BKIN/TIM3_CH1/PA6)
- net BT_9_PA7: now also P9.4 (P4), U1.23 (ADC1_IN7/I2S1_SD/SPI1_MOSI/TIM1_CH1N/TIM3_CH2/PA7); no longer P9.3 (P3)
- net GND: now also R21.1, C27.2, D2.2 (A), R15.1
- net GNDA: now also R21.2
- net GPS_RX: now also P7.1 (P1), U1.42 (I2C3_SMBA/SDIO_D2/TIM1_CH2/USART1_TX/USB_OTG_FS_VBUS/PA9); no longer R21.2
- net IMU_I2C_CL: now also U1.61 (I2C1_SCL/I2C3_SDA/I2S5_SD/SDIO_D4/SPI5_MOSI/TIM10_CH1/TIM4_CH3/PB8); no longer U1.58 (I2C1_SCL/TIM4_CH1/USART1_TX/PB6)
- net IMU_I2C_DA: now also U1.62 (I2C1_SDA/I2C2_SDA/I2S2_WS/SDIO_D5/SPI2_NSS/TIM11_CH1/TIM4_CH4/PB9); no longer U1.59 (I2C1_SDA/SDIO_D0/TIM4_CH2/USART1_RX/PB7)
- net LSM6DSL_INT1: now also U1.56 (I2C3_SDA/I2S3_ext_SD/SDIO_D0/SPI1_MISO/SPI3_MISO/SYS_JTRST/TIM3_CH1/PB4)
- net LSM6DSL_INT2: now also U1.57 (I2C1_SMBA/I2S1_SD/I2S3_SD/SDIO_D3/SPI1_MOSI/SPI3_MOSI/TIM3_CH2/PB5)
- net PC13: now reaches U1.2 (PC13/ANTI_TAMP/RTC_AF1)
- net PC13: now also C27.1, R18.1, U8.1
- net 303C_I_XL: now reaches U1.20 (ADC1_IN4/I2S1_WS/I2S3_WS/SPI1_NSS/SPI3_NSS/USART2_CK/PA4)
- net 303C_I_XL: now also P12.2 (P2), U6.12 (INT_XL)
- net 303C_I_MAG: now reaches U1.21 (ADC1_IN5/I2S1_CK/SPI1_SCK/TIM2_CH1/TIM2_ETR/PA5)
- net 303C_DRDY: now reaches U1.26 (ADC1_IN8/I2S5_CK/SPI5_SCK/TIM1_CH2N/TIM3_CH3/PB0)
- net 303C_DRDY: now also P12.3 (P3), U6.11 (DRDY_MAG)
- removed net GPS_USART_TX: P7.1 (P1), R21.1, U1.42 (I2C3_SMBA/SDIO_D2/TIM1_CH2/USART1_TX/USB_OTG_FS_VBUS/PA9)
- removed net LSM303AGR_INT_1_XL: P12.3 (P3), U6.12 (INT_1_XL)
- removed net LSM303AGR_INT_2_XL: P12.2 (P2), U6.11 (INT_2_XL)
- new net: R15.2, U8.2
- no-connect marks 75 -> 63
Other:
- note added: "GP Button."
