File: Hardware/CPU_Board/CPU_Board.sch (KiCad schematic (older format))
At the start: 91 parts, among them P1 CONN_01X02, P10 CONN_01X03, P11 CONN_01X01, P12 CONN_01X03, P13 CONN_01X01, P14 CONN_01X03, P15 CONN_01X01, P16 CONN_01X01, P17 CONN_01X01, P18 CONN_01X01, P19 CONN_01X01, P2 USB_B, P20 CONN_01X01, P3 CONN_01X04, P4 CONN_01X06, P5 CONN_01X02, P6 CONN_01X02, P7 CONN_01X02, P8 CONN_01X02, P9 CONN_01X06, Q1 Q_PMOS_GSD, Q2 Q_PNP_BCE, Q3 Q_PNP_BCE, Q4 N-Channel, Q5 P-Channel, U1 STM32F411RETx, U2 FT232RL, U3 LM1117ADJ, U4 SPBTLE-RF, U5 A2235-H, U6 LSM303AGR, U7 LSM6DSL, U8 MCDTS2-4N, U9 INA128, Y1 8MHz

Commit message: Ready to manufacture!
Other:
- note added: "Reset\nSPI_MISO\nSPI_CLK\nSPI_MOSI\nSPI_CS\nSPI_IRQ"
- note removed: "Reset\nSPI_MISO\nSPI_MOSI\nSPI_CLK\nSPI_CS\nSPI_IRQ"
Changed lines of the file:
@@
 BT_5_PA0
 Text Notes 17000 7200 0    60   ~ 0
-Reset\nSPI_MISO\nSPI_MOSI\nSPI_CLK\nSPI_CS\nSPI_IRQ
+Reset\nSPI_MISO\nSPI_CLK\nSPI_MOSI\nSPI_CS\nSPI_IRQ
 $Comp
 L CONN_01X06 P9
