File: Hardware/CPU_Board/CPU_Board.kicad_pcb (KiCad board)
At the start: 2 copper layers, 76 parts, among them P1 CONN_01X02, P10 CONN_01X04, P2 USB_B, P3 CONN_01X06, P4 CONN_01X01, P5 CONN_01X01, P6 CONN_01X01, P7 CONN_01X01, P8 CONN_01X01, P9 CONN_01X01, Q1 Q_PMOS_GSD, Q2 Q_PNP_BCE, Q3 Q_PNP_BCE, Q4 N-Channel, Q5 P-Channel, U1 STM32F411RETx, U2 FT232RL, U3 LM1117ADJ, U4 6N136, U5 SPBTLE-RF, U6 A2235-H, U7 LSM303AGR, U8 LSM6DSL, U9 INA128, Y1 8MHz

Commit message: PCB v0.1.0
* Changed components to SMD
* Added Measurement nodes for all datalines
* Designed PCB (Rather big now, only a first edition!)
* "Fixed" fucked up power flags
Parts:
- removed C30: 100nF, Capacitors_ThroughHole:C_Axial_L3.8mm_D2.6mm_P7.50mm_Horizontal
- removed the U4 at (272.4, 128.4)
- removed the U6 at (250.5, 74.0)
- added C22: 100n, Capacitors_SMD:C_0805_HandSoldering, F.Cu at (144.5, 120.4)
- added P10: CONN_01X03, Pin_Headers:Pin_Header_Straight_1x03_Pitch2.54mm, F.Cu at (30.7, 168.1)
- added P11: CONN_01X01, Pin_Headers:Pin_Header_Straight_1x01_Pitch2.54mm, F.Cu at (113.0, 127.8)
- added P12: CONN_01X03, Pin_Headers:Pin_Header_Straight_1x03_Pitch2.54mm, F.Cu at (126.6, 100.2)
- added P13: CONN_01X01, Pin_Headers:Pin_Header_Straight_1x01_Pitch2.54mm, F.Cu at (45.3, 119.5)
- added P14: CONN_01X03, Pin_Headers:Pin_Header_Straight_1x03_Pitch2.54mm, F.Cu at (55.1, 134.6)
- added P5: CONN_01X02, Pin_Headers:Pin_Header_Straight_1x02_Pitch2.54mm, F.Cu at (108.6, 100.5)
- added P6: CONN_01X02, Pin_Headers:Pin_Header_Straight_1x02_Pitch2.54mm, F.Cu at (66.0, 102.2)
- added P7: CONN_01X02, Pin_Headers:Pin_Header_Straight_1x02_Pitch2.54mm, F.Cu at (113.0, 118.1)
- added P8: CONN_01X02, Pin_Headers:Pin_Header_Straight_1x02_Pitch2.54mm, F.Cu at (102.4, 93.5)
- added P9: CONN_01X06, Pin_Headers:Pin_Header_Straight_1x06_Pitch2.54mm, F.Cu at (98.4, 147.2)
- added R19: 0C, Resistors_ThroughHole:R_Axial_DIN0204_L3.6mm_D1.6mm_P1.90mm_Vertical, F.Cu at (114.3, 123.9)
- added R20: 0C, Resistors_ThroughHole:R_Axial_DIN0204_L3.6mm_D1.6mm_P2.54mm_Vertical, F.Cu at (117.3, 121.3)
- added R21: 0C, Resistors_ThroughHole:R_Axial_DIN0204_L3.6mm_D1.6mm_P1.90mm_Vertical, F.Cu at (117.3, 118.1)
- added R22: 0C, Resistors_ThroughHole:R_Axial_DIN0204_L3.6mm_D1.6mm_P1.90mm_Vertical, F.Cu at (119.8, 120.5)
- added U5: A2235-H, FOOTPRINTS:A2235-H_Handsolder, F.Cu at (125.3, 131.9)
- C1, C10, C12, C14, C15, C16, C18, C2, C20, C27, C28, C3, C6, C8: footprint Capacitors_ThroughHole:C_Axial_L3.8mm_D2.6mm_P7.50mm_Horizontal -> Capacitors_SMD:C_0805_HandSoldering
- C11: value 4.7u -> 100n; footprint Capacitors_ThroughHole:CP_Axial_L10.0mm_D4.5mm_P15.00mm_Horizontal -> Capacitors_SMD:C_0805_HandSoldering
- C13: value 10u -> 100n; footprint Capacitors_ThroughHole:CP_Axial_L10.0mm_D4.5mm_P15.00mm_Horizontal -> Capacitors_SMD:C_0805_HandSoldering
- C17: value 100n -> 10u; footprint Capacitors_ThroughHole:C_Axial_L3.8mm_D2.6mm_P7.50mm_Horizontal -> Capacitors_SMD:CP_Elec_5x5.3
- C19, C7: footprint Capacitors_ThroughHole:CP_Axial_L10.0mm_D4.5mm_P15.00mm_Horizontal -> Capacitors_SMD:CP_Elec_5x5.3
- C21: value 100n -> 1uF; footprint Capacitors_ThroughHole:C_Axial_L3.8mm_D2.6mm_P7.50mm_Horizontal -> Capacitors_SMD:C_0805_HandSoldering
- C23: value 1uF -> 220nF; footprint Capacitors_ThroughHole:C_Axial_L3.8mm_D2.6mm_P7.50mm_Horizontal -> Capacitors_SMD:C_0805_HandSoldering
- C24: value 100n -> 10uF; footprint Capacitors_ThroughHole:C_Axial_L3.8mm_D2.6mm_P7.50mm_Horizontal -> Capacitors_SMD:CP_Elec_5x5.3
- C25: value 220nF -> 100nF; footprint Capacitors_ThroughHole:C_Axial_L3.8mm_D2.6mm_P7.50mm_Horizontal -> Capacitors_SMD:C_0805_HandSoldering
- C26: value 10uF -> 100nF; footprint Capacitors_ThroughHole:CP_Axial_L10.0mm_D4.5mm_P15.00mm_Horizontal -> Capacitors_SMD:C_0805_HandSoldering
- C29: value 100nF -> 100n; footprint Capacitors_ThroughHole:C_Axial_L3.8mm_D2.6mm_P7.50mm_Horizontal -> Capacitors_SMD:C_0805_HandSoldering
- C4, C5: footprint Capacitors_ThroughHole:CP_Axial_L10.0mm_D4.5mm_P15.00mm_Horizontal -> Capacitors_SMD:CP_Elec_4x5.3
- C9: value 100n -> 4.7u; footprint Capacitors_ThroughHole:C_Axial_L3.8mm_D2.6mm_P7.50mm_Horizontal -> Capacitors_SMD:CP_Elec_4x5.3
- D1: footprint Diodes_ThroughHole:D_5W_P5.08mm_Vertical_AnodeUp -> Diodes_SMD:D_SOD-323
- L2, L3: footprint Connectors:bornier2 -> Inductors:INDUCTOR_V
- R1, R10, R11, R12, R13, R15, R16, R17, R18, R2, R3, R4, R5, R6, R7, R8, R9: footprint Resistors_ThroughHole:R_Axial_DIN0204_L3.6mm_D1.6mm_P5.08mm_Horizontal -> Resistors_SMD:R_0805_HandSoldering
- moved R6 172.8 mm to (101.3, 157.3), turned to 180 degrees
- moved R9 167.9 mm to (101.3, 159.2), turned to 180 degrees
- moved C24 155.7 mm to (121.1, 98.2)
- moved C23 147.5 mm to (113.6, 102.4)
- moved Q4 146.9 mm to (115.7, 132.8), turned to 180 degrees
- moved Q5 146.6 mm to (110.2, 132.8)
- moved U4 146.1 mm to (111.8, 155.7), turned to 180 degrees
- moved R7 145.8 mm to (144.6, 125.3)
- moved R14 138.4 mm to (117.9, 127.8)
- moved R8 137.9 mm to (144.5, 115.7), turned to 270 degrees
- moved R16 136.6 mm to (120.3, 127.8), turned to 90 degrees
- moved C11 134.9 mm to (63.9, 165.0), turned to 270 degrees
- moved R11 133.5 mm to (132.0, 112.4), turned to 180 degrees
- moved R15 131.1 mm to (122.7, 129.1)
- moved R18 129.3 mm to (121.6, 134.3)
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- renumbered P4 to P15, P5 to P16, P6 to P17, P7 to P18, P8 to P19, P9 to P20, P10 to P3, P3 to P4, U5 to U4, U7 to U6, U8 to U7, U9 to U8
Connections:
- C10 pad 1: Net-(C10-Pad1) -> GND
- C10 pad 2: GND -> +3V3
- C11 pad 1: +3V3 -> Net-(C11-Pad1)
- C12 pad 1: +5VA -> GND
- C12 pad 2: GNDA -> +3V3
- C13 pad 1: Net-(C10-Pad1) -> Net-(C11-Pad1)
- C16 pad 1: GND -> +5VA
- C16 pad 2: +3V3 -> GNDA
- C17 pad 1: GND -> Net-(C11-Pad1)
- C17 pad 2: +3V3 -> GND
- C21 pad 1: GND -> +3V3
- C21 pad 2: +3V3 -> GND
- C23 pad 1: +3V3 -> Net-(C23-Pad1)
- C25 pad 1: Net-(C25-Pad1) -> +3V3
- C29 pad 1: +3V3 -> GND
- C29 pad 2: GND -> +3V3
- C9 pad 1: Net-(C10-Pad1) -> +3V3
- L2 pad 2: Net-(C10-Pad1) -> Net-(C11-Pad1)
- P2 pad 1: GND -> Net-(L1-Pad1)
- P2 pad 4: Net-(L1-Pad1) -> GND
- P2 pad 5: Net-(P2-Pad5) -> GND
- Q3 pad 2: Net-(C10-Pad1) -> Net-(C11-Pad1)
- U1 pad 24: (no net) -> /Load_cell_amp
- U1 pad 25: (no net) -> GNDA
- U1 pad 41: /IMU_I2C_CL -> (no net)
- U1 pad 42: (no net) -> /GPS_USART_TX
- U1 pad 43: (no net) -> /GPS_USART_RX
- U1 pad 56: /IMU_I2C_DA -> (no net)
- U1 pad 58: (no net) -> /IMU_I2C_CL
- U1 pad 59: (no net) -> /IMU_I2C_DA
- U1 pad 8: /Load_cell_amp -> (no net)
- U2 pad 15: Net-(P2-Pad2) -> Net-(P2-Pad3)
- U2 pad 16: Net-(P2-Pad3) -> Net-(P2-Pad2)
- U3 pad 3: Net-(C10-Pad1) -> Net-(C11-Pad1)
- U4 pad 7: (no net) -> /BT_7_PB3
- U4 pad 8: (no net) -> /BT_8_PA6
- U4 pad 9: (no net) -> /BT_9_PA7
- U6 pad 11: (no net) -> /LSM303AGR_INT_2_XL
- U6 pad 12: (no net) -> /LSM303AGR_INT_1_XL
- U6 pad 5: Net-(C25-Pad1) -> Net-(C23-Pad1)
- U6 pad 7: (no net) -> /LSM303AGR_INT_MAG
- U7 pad 4: (no net) -> /LSM6DSL_INT1
- U7 pad 9: (no net) -> /LSM6DSL_INT2
Routing:
- net GND: track 0.00 -> 560.9 mm, vias 0 -> 15
- net +3V3: track 0.00 -> 511.3 mm, vias 0 -> 10
- net GNDA: track 0.00 -> 83.6 mm
- net +5VA: track 0.00 -> 52.1 mm
- net /Load_cell_amp: track 0.00 -> 51.5 mm
- net /IMU_I2C_CL: track 0.00 -> 51.3 mm, vias 0 -> 1
- net /SWCLK: track 0.00 -> 46.2 mm, vias 0 -> 1
- net Net-(C11-Pad1): track 0.00 -> 43.7 mm
- net /SWDIO: track 0.00 -> 41.9 mm, vias 0 -> 1
- net /IMU_I2C_DA: track 0.00 -> 39.7 mm, vias 0 -> 1
- net Net-(Q4-Pad2): track 0.00 -> 37.4 mm
- net /USB_USART_TX: track 0.00 -> 36.2 mm
- net /GPS_USART_RX: track 0.00 -> 33.7 mm
- net /USB_USART_RX: track 0.00 -> 33.5 mm
- net /GPS_USART_TX: track 0.00 -> 29.7 mm
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- added copper zone on B.Cu, net GND
- added copper zone on F.Cu, net GND
- added copper zone on B.Cu, net GNDA
- added copper zone on F.Cu, net GNDA
Other:
- board outline added: 272.7 x 170.7 mm
- rule trace_min: 0.2 -> 0.15
- rule via_min_size: 0.4 -> 0.35
- board text added: "303 INT1 303 INT2 303 INT"
- board text added: "3V3"
- board text added: "Analog"
- board text added: "BT"
- board text added: "CL DA"
- board text added: "CLK DIO"
- board text added: "G"
- board text added: "GPS"
- board text added: "I2 I1"
- board text added: "NRST"
- board text added: "Power"
- board text added: "R MI MO CL CS IRQ"
- board text added: "SailorAid"
- board text added: "TOG"
- board text added: "TX RX"
- board text added: "USB"

Commit message: Small PCB update and Manufacturing
* CPU_Board v0.1.1
* Manufacturing files (Gerbers, mapping, drill etc.)
Parts:
- moved P19 220.0 mm to (75.8, 133.5)
- moved P20 154.1 mm to (142.4, 92.7)
- moved P16 153.3 mm to (92.5, 165.7)
- moved P15 88.9 mm to (30.6, 110.2)
- moved P18 40.3 mm to (132.3, 147.7)
- moved P17 30.7 mm to (30.6, 146.1)
Changed lines of the file:
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@@
     (links 215)
     (no_connects 0)
-    (area 24.399993 -0.075096 297.255001 210.133001)
+    (area 22.007 -0.075001 297.255001 191.975)
     (thickness 1.6)
     (drawings 27)
@@
     (0 F.Cu signal)
     (31 B.Cu signal)
-    (32 B.Adhes user)
-    (33 F.Adhes user)
-    (34 B.Paste user)
-    (35 F.Paste user)
-    (36 B.SilkS user)
+    (32 B.Adhes user hide)
+    (33 F.Adhes user hide)
+    (34 B.Paste user hide)
+    (35 F.Paste user hide)
+    (36 B.SilkS user hide)
     (37 F.SilkS user)
-    (38 B.Mask user)
-    (39 F.Mask user)
-    (40 Dwgs.User user)
-    (41 Cmts.User user)
-    (42 Eco1.User user)
-    (43 Eco2.User user)
-    (44 Edge.Cuts user)
-    (45 Margin user)
-    (46 B.CrtYd user)
-    (47 F.CrtYd user)
-    (48 B.Fab user)
-    (49 F.Fab user)
+    (38 B.Mask user hide)
+    (39 F.Mask user hide)
+    (40 Dwgs.User user hide)
+    (41 Cmts.User user hide)
+    (42 Eco1.User user hide)
+    (43 Eco2.User user hide)
+    (44 Edge.Cuts user hide)
+    (45 Margin user hide)
+    (46 B.CrtYd user hide)
+    (47 F.CrtYd user hide)
+    (48 B.Fab user hide)
+    (49 F.Fab user hide)
   )
   (setup
-    (last_trace_width 0.3)
+    (last_trace_width 0.25)
     (user_trace_width 0.15)
     (user_trace_width 0.2)
@@
   )
   (module Mounting_Holes:MountingHole_2.2mm_M2_DIN965_Pad (layer F.Cu)
-    (at 36.5 21.5)
+    (at 30.59 110.18)
     (descr "Mounting Hole 2.2mm, M2, DIN965")
     (tags "mounting hole 2.2mm m2 din965")
@@
   )
   (module Mounting_Holes:MountingHole_2.2mm_M2_DIN965_Pad (layer F.Cu)
-    (at 151 24)
+    (at 92.45 165.66)
     (descr "Mounting Hole 2.2mm, M2, DIN965")
     (tags "mounting hole 2.2mm m2 din965")
@@
   )
   (module Mounting_Holes:MountingHole_2.2mm_M2_DIN965_Pad (layer F.Cu)
-    (at 29.23 176.784)
+    (at 30.61 146.13)
     (descr "Mounting Hole 2.2mm, M2, DIN965")
     (tags "mounting hole 2.2mm m2 din965")
@@
   )
   (module Mounting_Holes:MountingHole_2.2mm_M2_DIN965_Pad (layer F.Cu)
-    (at 141.5 187)
+    (at 132.35 147.74)
     (descr "Mounting Hole 2.2mm, M2, DIN965")
     (tags "mounting hole 2.2mm m2 din965")
@@
   )
   (module Mounting_Holes:MountingHole_2.2mm_M2_DIN965_Pad (layer F.Cu)
-    (at 266 23)
+    (at 75.78 133.52)
     (descr "Mounting Hole 2.2mm, M2, DIN965")
     (tags "mounting hole 2.2mm m2 din965")
@@
   )
   (module Mounting_Holes:MountingHole_2.2mm_M2_DIN965_Pad (layer F.Cu)
-    (at 263.5 188)
+    (at 142.38 92.68)
     (descr "Mounting Hole 2.2mm, M2, DIN965")
     (tags "mounting hole 2.2mm m2 din965")
-    (fp_text reference P20 (at 0 -2.9) (layer F.SilkS)
+    (fp_text reference P20 (at 0.13 -2.03) (layer F.SilkS)
       (effects (font (size 1 1) (thickness 0.15)))
     )
@@
     (descr "SMT capacitor, aluminium electrolytic, 5x5.3")
     (attr smd)
-    (fp_text reference C7 (at 0 3.92 180) (layer F.SilkS)
-      (effects (font (size 1 1) (thickness 0.15)))
-    )
+    (fp_text reference C7 (at 0.005 0.67 180) (layer F.SilkS)
+      (effects (font (size 1 1) (thickness 0.15)))
+    )

Commit message: PCB_Design v0.2
Added, changed and stuff.
Libraries and stuff.
Looks like shit, but it should work.
Will check later and then send gerbers.
Parts:
- removed the R19 at (114.3, 123.9)
- removed the R20 at (117.3, 121.3)
- removed R22: 0C, Resistors_ThroughHole:R_Axial_DIN0204_L3.6mm_D1.6mm_P1.90mm_Vertical
- added C27: 100n, Capacitors_SMD:C_0805_HandSoldering, F.Cu at (70.1, 131.1)
- added D2: D_Photo, Opto-Devices:PhotoDiode_SFH205, F.Cu at (81.8, 160.8)
- added R15: 1k, Resistors_SMD:R_0805_HandSoldering, F.Cu at (70.0, 135.6)
- added R18: 10k, Resistors_SMD:R_0805_HandSoldering, F.Cu at (75.0, 128.6)
- added U8: MCDTS2-4N, Buttons_Switches_SMD:SW_SPST_PTS645, F.Cu at (77.6, 133.3)
- R21: value 0C -> 0R; footprint Resistors_ThroughHole:R_Axial_DIN0204_L3.6mm_D1.6mm_P1.90mm_Vertical -> Resistors_ThroughHole:R_Axial_DIN0204_L3.6mm_D1.6mm_P5.08mm_Horizontal
- moved R21 87.0 mm to (34.0, 143.3), turned to 90 degrees
- moved P19 22.6 mm to (91.0, 150.2)
- moved P7 6.90 mm to (119.4, 115.3)
- moved R2 1.99 mm to (106.7, 117.6)
- moved C12 1.08 mm to (104.6, 116.1)
- moved P20 0.96 mm to (143.0, 91.9)
- moved C14 0.52 mm to (86.6, 118.1)
- renumbered C11 to C10, C10 to C11, C16 to C15, C15 to C16, C27 to C28, C28 to C29, C29 to C30, R15 to R16, R16 to R17, R17 to R19, R18 to R20, U8 to U9
Connections:
- P12 pad 1: /LSM303AGR_INT_MAG -> /303C_I_MAG
- P12 pad 2: /LSM303AGR_INT_2_XL -> /303C_I_XL
- P12 pad 3: /LSM303AGR_INT_1_XL -> /303C_DRDY
- P7 pad 1: /GPS_USART_TX -> /GPS_RX
- P7 pad 2: /GPS_USART_RX -> /GPS_TX
- P9 pad 3: /BT_9_PA7 -> /BT_7_PB3
- P9 pad 4: /BT_7_PB3 -> /BT_9_PA7
- R21 pad 1: /GPS_USART_TX -> GND
- R21 pad 2: /GPS_RX -> GNDA
- U1 pad 14: (no net) -> /BT_5_PA0
- U1 pad 15: (no net) -> /BT_10_PA1
- U1 pad 2: (no net) -> /PC13
- U1 pad 20: (no net) -> /303C_I_XL
- U1 pad 21: (no net) -> /303C_I_MAG
- U1 pad 22: (no net) -> /BT_8_PA6
- U1 pad 23: (no net) -> /BT_9_PA7
- U1 pad 26: (no net) -> /303C_DRDY
- U1 pad 41: (no net) -> /BT_11_PA8
- U1 pad 42: /GPS_USART_TX -> /GPS_RX
- U1 pad 43: /GPS_USART_RX -> /GPS_TX
- U1 pad 55: (no net) -> /BT_7_PB3
- U1 pad 56: (no net) -> /LSM6DSL_INT1
- U1 pad 57: (no net) -> /LSM6DSL_INT2
- U1 pad 58: /IMU_I2C_CL -> (no net)
- U1 pad 59: /IMU_I2C_DA -> (no net)
- U1 pad 61: (no net) -> /IMU_I2C_CL
- U1 pad 62: (no net) -> /IMU_I2C_DA
- U6 pad 11: /LSM303AGR_INT_2_XL -> /303C_DRDY
- U6 pad 12: /LSM303AGR_INT_1_XL -> /303C_I_XL
- U6 pad 7: /LSM303AGR_INT_MAG -> /303C_I_MAG
Routing:
- net /303C_DRDY: track 0.00 -> 80.6 mm, vias 0 -> 1
- net /303C_I_XL: track 0.00 -> 74.4 mm, vias 0 -> 1
- net /303C_I_MAG: track 0.00 -> 63.6 mm, vias 0 -> 1
- net /PC13: track 0.00 -> 44.7 mm, vias 0 -> 2
- net /BT_5_PA0: track 17.8 -> 60.1 mm, vias 0 -> 2
- net /BT_10_PA1: track 15.2 -> 56.2 mm, vias 0 -> 2
- net /LSM6DSL_INT2: track 8.11 -> 47.5 mm, vias 1 -> 2
- net /LSM6DSL_INT1: track 7.00 -> 46.2 mm, vias 0 -> 1
- net /BT_8_PA6: track 10.5 -> 45.3 mm, vias 0 -> 2
- net /BT_9_PA7: track 11.9 -> 46.6 mm, vias 0 -> 2
- net /GPS_USART_RX: track 33.7 -> 0.00 mm
- net /BT_11_PA8: track 17.1 -> 47.0 mm
- net /GPS_USART_TX: track 29.7 -> 0.00 mm
- net +3V3: track 511.3 -> 539.7 mm
- net /GPS_RX: track 17.4 -> 41.3 mm
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Other:
- board text added: "303 DRDY 303 IXL 303 IMAG"
- board text added: "R MI CL MO CS IRQ"
- board text removed: "303 INT1 303 INT2 303 INT"
- board text removed: "R MI MO CL CS IRQ"

Commit message: Ready to manufacture!
Parts:
- moved C16 0.90 mm to (87.8, 125.7)
- moved C5 0.13 mm to (84.3, 124.8)
Routing:
- net GND: track 572.3 -> 589.5 mm, vias 18 -> 22
- net +3V3: track 539.7 -> 554.1 mm, vias 10 -> 11
- net /IMU_I2C_CL: track 51.3 -> 47.9 mm
- net /BT_10_PA1: track 56.2 -> 59.3 mm
- net /BT_5_PA0: track 60.1 -> 63.2 mm
- net /BT_9_PA7: track 46.6 -> 49.2 mm
- net Net-(C5-Pad1): track 6.82 -> 5.67 mm
